File: hardware/fortunelabs_mainboard_v0/fortunelabs_mainboard_v0.kicad_sch (KiCad schematic)
At the start: 88 parts, among them J1 Conn_02x16_Odd_Even, J2 Conn_02x16_Odd_Even, J3 USB_C_Receptacle_USB2.0_14P, J4 SD_Card_Receptacle, J5 Conn_02x07_Odd_Even, Q1 AO3401A, SW1 BOOT, SW2 RESET, U1 ADS1115, U2 MCP23017_ML, U3 ESP32-S3-WROOM-2, U4 ADS1115, U5 TPS62162DSG, U6 DS3232M, U7 TPL5010, U8 ULN2803A

Commit message: add LICENSE
Parts:
- BT1: footprint CR2032 -> Battery:BatteryHolder_Keystone_3002_1x2032
Connections:
- net AGND is gone; now on net GND: J1.22 (Pin_22)
- net AVDD_3V3 is gone; now on net +3V3: J1.21 (Pin_21)
- net ESP32_GPIO is gone; now on net MCP_ESP32_GPIO: J1.29 (Pin_29)
- net +3V3: no longer J5.1 (Pin_1), J5.2 (Pin_2), J5.3 (Pin_3), J5.4 (Pin_4), J5.5 (Pin_5), J5.6 (Pin_6), J5.7 (Pin_7), J5.8 (Pin_8), R20.2, U3.10 (IO17), U8.11 (O8), U8.12 (O7), U8.13 (O6), U8.14 (O5), U8.15 (O4), U8.16 (O3), U8.17 (O2), U8.18 (O1)
- net GND: now also U1.1 (ADDR); no longer D10.1 (K), D2.1 (K), D4.1 (K), D5.1 (K), D6.1 (K), D7.1 (K), D8.1 (K), D9.1 (K)
- net MCP_ESP32_GPIO: now reaches U3.23 (IO21)
- new net OUT1: D10.1 (K), J5.1 (Pin_1), U8.18 (O1)
- new net OUT2: D9.1 (K), J5.3 (Pin_3), U8.17 (O2)
- new net OUT3: D8.1 (K), J5.5 (Pin_5), U8.16 (O3)
- new net OUT4: D7.1 (K), J5.7 (Pin_7), U8.15 (O4)
- new net OUT5: D6.1 (K), J5.2 (Pin_2), U8.14 (O5)
- new net OUT6: D5.1 (K), J5.4 (Pin_4), U8.13 (O6)
- new net OUT7: D4.1 (K), J5.6 (Pin_6), U8.12 (O7)
- new net OUT8: D2.1 (K), J5.8 (Pin_8), U8.11 (O8)
- new net RTC_INT: R20.2, U3.10 (IO17)
- no-connect marks 13 -> 29
Other:
- moved on the sheet: C13, C14, C6, L1, R10, R17, R8, R9, U2, U5

Commit message: hw(hardware): put EN and BOOT on their own nets, off the 3V3 rail
SW2 (RESET) and SW1 (BOOT) each sat directly across +3V3 and GND, so
either button shorted the rail when pressed. C18 sat across the rail as
well, leaving EN with a pull-up and no delay capacitor.

EN is now R21 (10K to +3V3), C18 (100n to GND), SW2 to GND, and U7 pin 6.
BOOT is now R24 (10K to +3V3) and SW1 to GND on U3 pin 27. Neither switch
touches +3V3.

R23 is removed: it was a second 10K pull-up in parallel with R21, halving
the EN time constant against C18 for no gain. R21 stays because U7's RSTn
is open collector and requires it.

SW1's left pin is routed around R24 at y=144.78 to reach the IO0 side; the
EN and IO0 spans are split at each tap so the junctions bond wire
endpoints, which is how the connectivity is actually computed.

Also fills the placeholder values on R21 and C18.

ERC: 0 errors, 0 warnings.
Parts:
- removed R23: R, symbol Device:R
- C18: value C -> 100n
- R21: value R -> 10K
Connections:
- net +3V3: no longer SW1.1, SW2.2
- net ESP32_EN: now also SW2.2
- net at R24.1, U3.27 (IO0): now also SW1.1
Changed lines of the file:
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@@
 	)
 	(junction
-		(at 246.38 138.43)
-		(diameter 0)
-		(color 0 0 0 0)
-	)
-	(junction
 		(at 113.03 78.74)
 		(diameter 0)
@@
 	)
 	(junction
-		(at 191.77 125.73)
-		(diameter 0)
-		(color 0 0 0 0)
-	)
-	(junction
 		(at 77.47 60.96)
 		(diameter 0)
@@
 	)
 	(junction
-		(at 191.77 138.43)
-		(diameter 0)
-		(color 0 0 0 0)
-	)
-	(junction
 		(at 279.4 59.69)
 		(diameter 0)
@@
 	(wire
 		(pts
-			(xy 363.22 171.45) (xy 360.68 171.45)
+			(xy 170.18 138.43) (xy 185.42 138.43)
 		)
 		(stroke
@@
 	(wire
 		(pts
-			(xy 297.18 48.26) (xy 309.88 48.26)
+			(xy 185.42 138.43) (xy 191.77 138.43)
 		)
 		(stroke
@@
 	(wire
 		(pts
-			(xy 297.18 55.88) (xy 309.88 55.88)
+			(xy 191.77 138.43) (xy 210.82 138.43)
 		)
 		(stroke
@@
 	(wire
 		(pts
-			(xy 67.31 138.43) (xy 92.71 138.43)
+			(xy 191.77 138.43) (xy 191.77 144.78)
 		)
 		(stroke
@@
 	(wire
 		(pts
-			(xy 27.94 36.83) (xy 27.94 43.18)
+			(xy 236.22 138.43) (xy 237.49 138.43)
 		)
 		(stroke
@@
 	(wire
 		(pts
-			(xy 64.77 251.46) (xy 73.66 251.46)
+			(xy 237.49 138.43) (xy 238.76 138.43)
 		)
 		(stroke
@@
 	(wire
 		(pts
-			(xy 335.28 50.8) (xy 335.28 62.23)
+			(xy 248.92 138.43) (xy 248.92 144.78)
 		)
 		(stroke
@@
 	(wire
 		(pts
-			(xy 91.44 222.25) (xy 91.44 223.52)
+			(xy 248.92 144.78) (xy 237.49 144.78)
 		)
 		(stroke
@@
 	(wire
 		(pts
-			(xy 45.72 121.92) (xy 59.69 121.92)
+			(xy 237.49 144.78) (xy 237.49 138.43)
 		)
 		(stroke
@@
 		)
 	)
+	(junction
+		(at 185.42 138.43)
+		(diameter 0)
+		(color 0 0 0 0)
+	)
+	(junction
+		(at 191.77 138.43)
+		(diameter 0)
+		(color 0 0 0 0)
+	)
+	(junction
+		(at 237.49 138.43)
+		(diameter 0)
+		(color 0 0 0 0)
+	)
 	(wire
 		(pts
-			(xy 276.86 49.53) (xy 290.83 49.53)
+			(xy 363.22 171.45) (xy 360.68 171.45)
 		)
 		(stroke
@@
 	(wire
 		(pts
-			(xy 121.92 251.46) (xy 127 251.46)
+			(xy 297.18 48.26) (xy 309.88 48.26)
 		)
 		(stroke
@@
 	(wire
 		(pts
-			(xy 40.64 238.76) (xy 44.45 238.76)
+			(xy 297.18 55.88) (xy 309.88 55.88)
 		)
 		(stroke
@@
 	(wire
 		(pts
-			(xy 316.23 99.06) (xy 327.66 99.06)
+			(xy 67.31 138.43) (xy 92.71 138.43)
 		)
 		(stroke
@@
 	(wire
 		(pts
-			(xy 82.55 180.34) (xy 82.55 182.88)
+			(xy 27.94 36.83) (xy 27.94 43.18)
 		)
 		(stroke
@@
 	(wire
 		(pts
-			(xy 276.86 57.15) (xy 290.83 57.15)
+			(xy 64.77 251.46) (xy 73.66 251.46)
 		)
 		(stroke
@@
 	(wire
 		(pts
-			(xy 347.98 120.65) (xy 358.14 120.65)
+			(xy 335.28 50.8) (xy 335.28 62.23)
 		)
 		(stroke
@@
 	(wire
 		(pts
-			(xy 246.38 138.43) (xy 248.92 138.43)
+			(xy 91.44 222.25) (xy 91.44 223.52)
 		)
 		(stroke
@@
 	(wire
 		(pts
-			(xy 191.77 138.43) (xy 191.77 134.62)
+			(xy 45.72 121.92) (xy 59.69 121.92)
+		)
+		(stroke
+			(width 0)
+			(type default)
+		)
+	)
+	(wire
+		(pts
+			(xy 276.86 49.53) (xy 290.83 49.53)
+		)
+		(stroke
+			(width 0)
+			(type default)
+		)
+	)
+	(wire
+		(pts
+			(xy 121.92 251.46) (xy 127 251.46)
+		)
+		(stroke
+			(width 0)
+			(type default)
+		)
+	)
+	(wire
+		(pts
+			(xy 40.64 238.76) (xy 44.45 238.76)
+		)
+		(stroke
+			(width 0)
+			(type default)
+		)
+	)
+	(wire
+		(pts
+			(xy 316.23 99.06) (xy 327.66 99.06)
+		)
+		(stroke
+			(width 0)
+			(type default)
+		)
+	)
+	(wire
+		(pts
+			(xy 82.55 180.34) (xy 82.55 182.88)
+		)
+		(stroke
+			(width 0)
+			(type default)
+		)
+	)
+	(wire
+		(pts
+			(xy 276.86 57.15) (xy 290.83 57.15)
+		)
+		(stroke
+			(width 0)
+			(type default)
+		)
+	)
+	(wire
+		(pts
+			(xy 347.98 120.65) (xy 358.14 120.65)
 		)
 		(stroke
@@
 	(wire
 		(pts
-			(xy 191.77 127) (xy 191.77 125.73)
-		)
-		(stroke
-			(width 0)
-			(type default)
-		)
-	)
-	(wire
-		(pts
 			(xy 85.09 71.12) (xy 85.09 81.28)
 		)
@@
 	(wire
 		(pts
-			(xy 185.42 125.73) (xy 191.77 125.73)
-		)
-		(stroke
-			(width 0)
-			(type default)
-		)
-	)
-	(wire
-		(pts
 			(xy 33.02 251.46) (xy 26.67 251.46)
 		)
@@
 	(wire
 		(pts
-			(xy 191.77 138.43) (xy 191.77 144.78)
-		)
-		(stroke
-			(width 0)
-			(type default)
-		)
-	)
-	(wire
-		(pts
 			(xy 40.64 243.84) (xy 44.45 243.84)
 		)
@@
 	(wire
 		(pts
-			(xy 191.77 125.73) (xy 223.52 125.73)
-		)
-		(stroke
-			(width 0)
-			(type default)
-		)
-	)
-	(wire
-		(pts
 			(xy 43.18 44.45) (xy 43.18 45.72)
 		)
@@
 	(wire
 		(pts
-			(xy 236.22 138.43) (xy 238.76 138.43)
-		)
-		(stroke
-			(width 0)
-			(type default)
-		)
-	)
-	(wire
-		(pts
 			(xy 365.76 219.71) (xy 393.7 219.71)
 		)
@@
 	(wire
 		(pts
-			(xy 185.42 142.24) (xy 185.42 125.73)
+			(xy 185.42 142.24) (xy 185.42 138.43)
 		)
 		(stroke
@@
 	(wire
 		(pts
-			(xy 170.18 138.43) (xy 191.77 138.43)
-		)
-		(stroke
-			(width 0)
-			(type default)
-		)
-	)
-	(wire
-		(pts
 			(xy 130.81 60.96) (xy 130.81 67.31)
 		)
@@
 	(wire
 		(pts
-			(xy 191.77 138.43) (xy 210.82 138.43)
-		)
-		(stroke
-			(width 0)
-			(type default)
-		)
-	)
-	(wire
-		(pts
 			(xy 295.91 99.06) (xy 308.61 99.06)
 		)
@@
 			)
 		)
-		(property "Value" "R"
+		(property "Value" "10K"
 			(at 374.396 212.852 0)
 			(effects
@@
 			)
 		)
-		(property "Value" "C"
+		(property "Value" "100n"
 			(at 195.58 149.8599 0)
 			(effects
@@
 					(unit 1)
 				)
-			)
-		)
-	)
-	(symbol
-		(lib_id "Device:R")
-		(at 191.77 130.81 0)
-		(unit 1)
-		(exclude_from_sim no)
-		(in_bom yes)
-		(on_board yes)
-		(dnp no)
-		(fields_autoplaced yes)
-		(property "Reference" "R23"
-			(at 194.31 129.5399 0)
-			(effects
-				(font
-					(size 1.27 1.27)
-				)
-				(justify left)
-			)
-		)
-		(property "Value" "R"
-			(at 194.31 132.0799 0)
-			(effects
-				(font
-					(size 1.27 1.27)
-				)
-				(justify left)
-			)
-		)
-		(property "Footprint" ""
-			(at 189.992 130.81 90)
-			(effects
-				(font
-					(size 1.27 1.27)
-				)
-				(hide yes)
-			)
-		)
-		(property "Datasheet" "~"
-			(at 191.77 130.81 0)
-			(effects
-				(font
-					(size 1.27 1.27)
-				)
-				(hide yes)
-			)
-		)
-		(property "Description" "Resistor"
-			(at 191.77 130.81 0)
-			(effects
-				(font
-					(size 1.27 1.27)
-				)
-				(hide yes)
-			)
-		)
-		(pin "2"
-		)
-		(pin "1"
-		)
-		(instances
-			(project "fortunelabs_mainboard_v0"
-				(path "/1727eecb-65c8-4b57-aa8a-814f366e0831"
-					(reference "R23")
-					(unit 1)
-				)

Commit message: hw(hardware): assign footprints and correct L1 value to 2u2
Footprint assignment pass over the v0 schematic: 75 Footprint properties
set or corrected, leaving F1 and J4 outstanding.

L1 carried the value "2L2", which is not valid notation for henries
("2R2" reads as 2.2 ohms). Corrected to "2u2", matching the 2.2 uH the
TPS62162 application circuit calls for alongside C13 (10u) and C14 (22u).

U8 moves from the DIP-18 SMD-socket land pattern to SOIC-18W. The
orderable part is therefore the ULN2803ADW; the Value field still reads
ULN2803A and is left for a separate decision.
Parts:
- C1, C10, C11, C15, C17, C18, C2, C3, C4, C5, C6, C7, C8, C9: footprint (none) -> Capacitor_SMD:C_0201_0603Metric
- C12: footprint (none) -> Capacitor_SMD:CP_Elec_6.3x5.4
- C13, C14: footprint (none) -> Capacitor_SMD:C_0805_2012Metric
- C16: footprint (none) -> Capacitor_SMD:C_0603_1608Metric
- D1: footprint (none) -> Diode_SMD:D_SMA
- D10: footprint LED_SMD:LED_0805_2012Metric -> LED_SMD:LED_0603_1608Metric
- D2, D4, D5, D6, D7, D8, D9: footprint (none) -> LED_SMD:LED_0603_1608Metric
- D3: footprint (none) -> Diode_SMD:D_SOD-123
- J1, J2: footprint (none) -> Connector_PinHeader_1.27mm:PinHeader_2x16_P1.27mm_Vertical
- J3: footprint (none) -> Connector_USB:USB_C_Receptacle_GCT_USB4105-xx-A_16P_TopMnt_Horizontal
- J5: footprint (none) -> Connector_PinHeader_1.27mm:PinHeader_2x07_P1.27mm_Vertical
- L1: value 2L2 -> 2u2; footprint (none) -> Inductor_SMD:L_APV_ANR3012
- R1, R10, R11, R12, R13, R14, R15, R16, R17, R18, R19, R2, R20, R21, R22, R24, R3, R33, R34, R35, R36, R37, R38, R39, R4, R40, R5, R6, R7, R8, R9: footprint (none) -> Resistor_SMD:R_0201_0603Metric
- R25, R26, R27, R28, R29, R30, R31, R32: footprint (none) -> Resistor_SMD:R_0603_1608Metric
- SW1, SW2: footprint (none) -> Button_Switch_SMD:SW_Push_1P1T_NO_CK_KMR2
- U8: footprint (none) -> Package_SO:SOIC-18W_7.5x11.6mm_P1.27mm

Commit message: hw(hardware): move passives to 0603 and C16 to 1210
Every resistor and capacitor carried an imperial 0201 land pattern
(R_0201_0603Metric, 0.6x0.3mm). The metric suffix names the same part in
two systems and reads as 0603 at a glance, which is how the board ended
up there while the LEDs sat on imperial 0603. 0201 is not hand-solderable
and Phase 8 leaves self-soldering against an assembly service open, so
the first spin should not foreclose it.

31 resistors and 14 capacitors move to the imperial 0603 land patterns
already used by the LEDs.

C16 is 100u and no 0603 part of that value exists, so the sweep alone
would have left it impossible. It takes C_1210_3225Metric, where 100u
6.3V X5R is stocked, keeping the bulk on +3V3 for ESP32-S3 transmit
bursts. Value unchanged.

F1 and J4 remain without footprints. J4 is held for the microSD change.
Parts:
- C1, C10, C11, C15, C17, C18, C2, C3, C4, C5, C6, C7, C8, C9: footprint Capacitor_SMD:C_0201_0603Metric -> Capacitor_SMD:C_0603_1608Metric
- C16: footprint Capacitor_SMD:C_0603_1608Metric -> Capacitor_SMD:C_1210_3225Metric
- R1, R10, R11, R12, R13, R14, R15, R16, R17, R18, R19, R2, R20, R21, R22, R24, R3, R33, R34, R35, R36, R37, R38, R39, R4, R40, R5, R6, R7, R8, R9: footprint Resistor_SMD:R_0201_0603Metric -> Resistor_SMD:R_0603_1608Metric
Changed lines of the file:
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@@
 			)
 		)
-		(property "Footprint" "Capacitor_SMD:C_0201_0603Metric"
+		(property "Footprint" "Capacitor_SMD:C_0603_1608Metric"
 			(at 93.98 179.3748 0)
 			(effects
@@
 			)
 		)
-		(property "Footprint" "Capacitor_SMD:C_0201_0603Metric"
+		(property "Footprint" "Capacitor_SMD:C_0603_1608Metric"
 			(at 328.6252 69.85 0)
 			(effects
@@
 			)
 		)
-		(property "Footprint" "Capacitor_SMD:C_0201_0603Metric"
+		(property "Footprint" "Capacitor_SMD:C_0603_1608Metric"
 			(at 344.17 30.1752 0)
 			(effects
@@
 			)
 		)
-		(property "Footprint" "Capacitor_SMD:C_0201_0603Metric"
+		(property "Footprint" "Capacitor_SMD:C_0603_1608Metric"
 			(at 342.5952 69.85 0)
 			(effects
@@
 			)
 		)
-		(property "Footprint" "Resistor_SMD:R_0201_0603Metric"
+		(property "Footprint" "Resistor_SMD:R_0603_1608Metric"
 			(at 93.472 229.87 90)
 			(effects
@@
 			)
 		)
-		(property "Footprint" "Resistor_SMD:R_0201_0603Metric"
+		(property "Footprint" "Resistor_SMD:R_0603_1608Metric"
 			(at 89.662 229.87 90)
 			(effects
@@
 			)
 		)
-		(property "Footprint" "Capacitor_SMD:C_0201_0603Metric"
+		(property "Footprint" "Capacitor_SMD:C_0603_1608Metric"
 			(at 342.5952 120.65 0)
 			(effects
@@
 			)
 		)
-		(property "Footprint" "Capacitor_SMD:C_0201_0603Metric"
+		(property "Footprint" "Capacitor_SMD:C_0603_1608Metric"
 			(at 336.2452 120.65 0)
 			(effects
@@
 			)
 		)
-		(property "Footprint" "Capacitor_SMD:C_0201_0603Metric"
+		(property "Footprint" "Capacitor_SMD:C_0603_1608Metric"
 			(at 348.9452 120.65 0)
 			(effects
@@
 			)
 		)
-		(property "Footprint" "Resistor_SMD:R_0201_0603Metric"
+		(property "Footprint" "Resistor_SMD:R_0603_1608Metric"
 			(at 97.282 229.87 90)
 			(effects
@@
 			)
 		)
-		(property "Footprint" "Resistor_SMD:R_0201_0603Metric"
+		(property "Footprint" "Resistor_SMD:R_0603_1608Metric"
 			(at 104.902 229.87 90)
 			(effects
@@
 			)
 		)
-		(property "Footprint" "Resistor_SMD:R_0201_0603Metric"
+		(property "Footprint" "Resistor_SMD:R_0603_1608Metric"
 			(at 312.42 103.378 90)
 			(effects
@@
 			)
 		)
-		(property "Footprint" "Resistor_SMD:R_0201_0603Metric"
+		(property "Footprint" "Resistor_SMD:R_0603_1608Metric"
 			(at 181.102 27.94 90)
 			(effects
@@
 			)
 		)
-		(property "Footprint" "Resistor_SMD:R_0201_0603Metric"
+		(property "Footprint" "Resistor_SMD:R_0603_1608Metric"
 			(at 370.332 213.36 90)
 			(effects
@@
 			)
 		)
-		(property "Footprint" "Resistor_SMD:R_0201_0603Metric"
+		(property "Footprint" "Resistor_SMD:R_0603_1608Metric"
 			(at 312.42 100.838 90)
 			(effects
@@
 			)
 		)
-		(property "Footprint" "Capacitor_SMD:C_0201_0603Metric"
+		(property "Footprint" "Capacitor_SMD:C_0603_1608Metric"
 			(at 192.7352 152.4 0)
 			(effects
@@
 			)
 		)
-		(property "Footprint" "Resistor_SMD:R_0201_0603Metric"
+		(property "Footprint" "Resistor_SMD:R_0603_1608Metric"
 			(at 100.33 197.358 90)
 			(effects
@@
 			)
 		)
-		(property "Footprint" "Capacitor_SMD:C_0201_0603Metric"
+		(property "Footprint" "Capacitor_SMD:C_0603_1608Metric"
 			(at 336.2452 69.85 0)
 			(effects
@@
 			)
 		)
-		(property "Footprint" "Resistor_SMD:R_0201_0603Metric"
+		(property "Footprint" "Resistor_SMD:R_0603_1608Metric"
 			(at 242.57 140.208 90)
 			(effects
@@
 			)
 		)
-		(property "Footprint" "Capacitor_SMD:C_0201_0603Metric"
+		(property "Footprint" "Capacitor_SMD:C_0603_1608Metric"
 			(at 328.6252 120.65 0)
 			(effects
@@
 			)
 		)
-		(property "Footprint" "Resistor_SMD:R_0201_0603Metric"
+		(property "Footprint" "Resistor_SMD:R_0603_1608Metric"
 			(at 385.572 63.5 90)
 			(effects
@@
 			)
 		)
-		(property "Footprint" "Resistor_SMD:R_0201_0603Metric"
+		(property "Footprint" "Resistor_SMD:R_0603_1608Metric"
 			(at 101.092 229.87 90)
 			(effects
@@
 			)
 		)
-		(property "Footprint" "Resistor_SMD:R_0201_0603Metric"
+		(property "Footprint" "Resistor_SMD:R_0603_1608Metric"
 			(at 313.69 55.118 90)
 			(effects
@@
 			)
 		)
-		(property "Footprint" "Resistor_SMD:R_0201_0603Metric"
+		(property "Footprint" "Resistor_SMD:R_0603_1608Metric"
 			(at 313.69 50.038 90)
 			(effects
@@
 			)
 		)
-		(property "Footprint" "Resistor_SMD:R_0201_0603Metric"
+		(property "Footprint" "Resistor_SMD:R_0603_1608Metric"
 			(at 108.712 229.87 90)
 			(effects
@@
 			)
 		)
-		(property "Footprint" "Capacitor_SMD:C_0201_0603Metric"
+		(property "Footprint" "Capacitor_SMD:C_0603_1608Metric"
 			(at 344.17 80.9752 0)
 			(effects
@@
 			)
 		)
-		(property "Footprint" "Resistor_SMD:R_0201_0603Metric"
+		(property "Footprint" "Resistor_SMD:R_0603_1608Metric"
 			(at 46.482 138.43 90)
 			(effects
@@
 			)
 		)
-		(property "Footprint" "Resistor_SMD:R_0201_0603Metric"
+		(property "Footprint" "Resistor_SMD:R_0603_1608Metric"
 			(at 41.402 50.8 90)
 			(effects
@@
 			)
 		)
-		(property "Footprint" "Resistor_SMD:R_0201_0603Metric"
+		(property "Footprint" "Resistor_SMD:R_0603_1608Metric"
 			(at 49.022 138.43 90)
 			(effects
@@
 			)
 		)
-		(property "Footprint" "Capacitor_SMD:C_0201_0603Metric"
+		(property "Footprint" "Capacitor_SMD:C_0603_1608Metric"
 			(at 120.65 109.5248 0)
 			(effects
@@
 			)
 		)
-		(property "Footprint" "Resistor_SMD:R_0201_0603Metric"
+		(property "Footprint" "Resistor_SMD:R_0603_1608Metric"
 			(at 116.332 229.87 90)
 			(effects
@@
 			)
 		)
-		(property "Footprint" "Resistor_SMD:R_0201_0603Metric"
+		(property "Footprint" "Resistor_SMD:R_0603_1608Metric"
 			(at 313.69 52.578 90)
 			(effects
@@
 			)
 		)
-		(property "Footprint" "Capacitor_SMD:C_0201_0603Metric"
+		(property "Footprint" "Capacitor_SMD:C_0603_1608Metric"
 			(at 348.9452 69.85 0)
 			(effects
@@
 			)
 		)
-		(property "Footprint" "Resistor_SMD:R_0201_0603Metric"
+		(property "Footprint" "Resistor_SMD:R_0603_1608Metric"
 			(at 112.522 229.87 90)
 			(effects
@@
 			)
 		)
-		(property "Footprint" "Capacitor_SMD:C_0603_1608Metric"
+		(property "Footprint" "Capacitor_SMD:C_1210_3225Metric"
 			(at 120.65 104.4448 0)
 			(effects
@@
 			)
 		)
-		(property "Footprint" "Resistor_SMD:R_0201_0603Metric"
+		(property "Footprint" "Resistor_SMD:R_0603_1608Metric"
 			(at 188.722 27.94 90)
 			(effects
@@
 			)
 		)
-		(property "Footprint" "Resistor_SMD:R_0201_0603Metric"
+		(property "Footprint" "Resistor_SMD:R_0603_1608Metric"
 			(at 329.692 224.79 90)
 			(effects
@@
 			)
 		)
-		(property "Footprint" "Resistor_SMD:R_0201_0603Metric"
+		(property "Footprint" "Resistor_SMD:R_0603_1608Metric"
 			(at 312.42 105.918 90)
 			(effects
@@
 			)
 		)
-		(property "Footprint" "Resistor_SMD:R_0201_0603Metric"
+		(property "Footprint" "Resistor_SMD:R_0603_1608Metric"
 			(at 118.872 71.12 90)
 			(effects
@@
 			)
 		)
-		(property "Footprint" "Resistor_SMD:R_0201_0603Metric"
+		(property "Footprint" "Resistor_SMD:R_0603_1608Metric"
 			(at 391.668 100.33 90)
 			(effects
@@
 			)
 		)
-		(property "Footprint" "Capacitor_SMD:C_0201_0603Metric"
+		(property "Footprint" "Capacitor_SMD:C_0603_1608Metric"
 			(at 187.6552 48.26 0)
 			(effects
@@
 			)
 		)
-		(property "Footprint" "Resistor_SMD:R_0201_0603Metric"
+		(property "Footprint" "Resistor_SMD:R_0603_1608Metric"
 			(at 313.69 57.658 90)
 			(effects
@@
 			)
 		)
-		(property "Footprint" "Resistor_SMD:R_0201_0603Metric"
+		(property "Footprint" "Resistor_SMD:R_0603_1608Metric"
 			(at 312.42 108.458 90)
 			(effects
@@
 			)
 		)
-		(property "Footprint" "Resistor_SMD:R_0201_0603Metric"
+		(property "Footprint" "Resistor_SMD:R_0603_1608Metric"
 			(at 177.292 44.45 90)
 			(effects
@@
 			)
 		)
-		(property "Footprint" "Resistor_SMD:R_0201_0603Metric"
+		(property "Footprint" "Resistor_SMD:R_0603_1608Metric"
 			(at 388.112 63.5 90)
 			(effects
@@
 			)
 		)
-		(property "Footprint" "Resistor_SMD:R_0201_0603Metric"
+		(property "Footprint" "Resistor_SMD:R_0603_1608Metric"
 			(at 383.032 63.5 90)
 			(effects

Commit message: hw(hardware): give F1 the 1812 polyfuse land pattern
F1 was the last component without a footprint apart from J4, which is
held for the microSD change. Fuse_1812_4532Metric is the common PPTC
land pattern in the 0.5A to 2A range this rail would use.

This assigns a package and nothing else. F1 remains electrically inert:
F1.1 sits on +12V and F1.2 reaches only D1.2 and Q1.3, a three-node net
that terminates there. The 12V supply enters on J5.13/14, already on the
+12V rail, so no current passes through the fuse, the TVS or the
reverse-polarity FET. That is a wiring defect and is owed its own issue.
Parts:
- F1: footprint (none) -> Fuse:Fuse_1812_4532Metric
Changed lines of the file:
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@@
 			)
 		)
-		(property "Footprint" ""
+		(property "Footprint" "Fuse:Fuse_1812_4532Metric"
 			(at 29.21 35.56 0)
 			(effects

Commit message: hw(hardware): rebuild the SD block around a microSD socket
J4 was a full-size SD receptacle: a 13-pin symbol with nine contacts,
a write-protect switch and two shell tabs. It becomes a Hirose DM3AT
microSD socket, symbol Micro_SD_Card_Det_Hirose_DM3AT with the matching
11-pad footprint.

The two symbols number their pins differently, so the block was rewired
rather than remapped. Only VDD, CLK, DAT0 and DAT1 keep their numbers;
SD_CS moves from pin 1 to pin 2, SD_MOSI from 2 to 3, DAT2 from 9 to 1,
and the shell tabs collapse from 12 and 13 onto pin 11. Nothing is lost:
write-protect and card-detect were already unconnected, and both VSS pins
were on GND, so the single VSS at pin 6 carries what two used to.

RN1 is replaced by five discrete 10K pull-ups on SD_CS, SD_MOSI, SD_MISO,
DAT1 and DAT2. It was an R_Network05 in a through-hole SIP6 array on an
otherwise surface-mount board, and its Value field still held the symbol
name, so no resistance had ever been assigned. CLK is left unpulled: it
is push-pull driven.

DET_A and DET_B are tied to GND. Card detect is not used.

SD_CS, SD_MOSI, SD_CLK and SD_MISO stay on IO10, IO11, IO12 and IO13,
which are the ESP32-S3 IOMUX pins for FSPI. The ESP32 side is untouched.

This leaves the schematic with no component lacking a footprint.
Parts:
- removed J4: SD_Card_Receptacle, symbol Connector:SD_Card_Receptacle
- removed RN1: R_Network05, Resistor_THT:R_Array_SIP6, symbol Device:R_Network05
- added J4: Micro_SD_Card_Det_Hirose_DM3AT, Connector_Card:microSD_HC_Hirose_DM3AT-SF-PEJM5, symbol Connector:Micro_SD_Card_Det_Hirose_DM3AT
- added R23, R41, R42, R43, R44: 10K, Resistor_SMD:R_0603_1608Metric, symbol Device:R
- C16: footprint Capacitor_SMD:C_1210_3225Metric -> Capacitor_SMD:C_0603_1608Metric
Connections:
- net +3V3: now also C15.2, C16.2, J4.4 (VDD), R23.1, R41.1, R42.1, R43.1, R44.1; no longer C15.1, C16.1
- net GND: now also C15.1, C16.1, J4.10 (DET_A), J4.11 (SHIELD), J4.6 (VSS), J4.9 (DET_B); no longer C15.2, C16.2
- net SD_CLK: now also J4.5 (CLK)
- net SD_CS: now also J4.2 (DAT3/CD), R43.2
- net SD_MISO: now also J4.7 (DAT0), R41.2
- net SD_MOSI: now also J4.3 (CMD), R42.2
- new net: J4.8 (DAT1), R23.2
- new net: J4.1 (DAT2), R44.2
- no-connect marks 29 -> 27
