File: hardware/fortunelabs_mainboard_v0/fortunelabs_mainboard_v0.kicad_sch (KiCad schematic)
At the start: 91 parts, among them J1 Conn_02x16_Odd_Even, J2 Conn_02x16_Odd_Even, J3 USB_C_Receptacle_USB2.0_14P, J4 Micro_SD_Card_Det_Hirose_DM3AT, J5 Conn_02x07_Odd_Even, Q1 AO3401A, SW1 BOOT, SW2 RESET, U1 ADS1115, U2 MCP23017_ML, U3 ESP32-S3-WROOM-2, U4 ADS1115, U5 TPS62162DSG, U6 DS3232M, U7 TPL5010, U8 ULN2803A

Commit message: hw(hardware): decouple the ESP32-S3 module supply pin
U3 (ESP32-S3-WROOM-2) pin 2 3V3 carried no local capacitor. The rail's
only reservoir was C14/C16 at the U5 buck output, shared with every
other device on +3V3.

Adds C19 100n 0603 and C20 22u 0805 at the 3V3 entry.

C19 satisfies the Phase 2.1 deliverable "0.1 uF decoupling cap at the
VDD of every IC". C20 is beyond that deliverable and is owed a
justification: ESP32-S3-WROOM-2 datasheet v1.7, section 9 Figure 9-1
Peripheral Schematics, shows 22 uF and 0.1 uF on VDD33 at the module
3V3 pin. The chip-level ESP32-S3 datasheet does not cover external
decoupling at all and cannot be cited for this.

Sizing rationale, from ESP32-S3 datasheet v2.2 Table 5-7 and 5-2:
peak TX 340 mA at 802.11b 21 dBm, and a recommended single-supply
output of 500 mA or more. U5 is a 1 A TPS62162, so supply capacity is
adequate; what was missing was the local reservoir for the RF bursts.

Whether this decouples anything in practice is a layout question and
is not settled here: the PCB carries no footprints yet.

ERC: 0 violations.
Parts:
- added C19: 100n, Capacitor_SMD:C_0603_1608Metric, symbol Device:C
- added C20: 22u, Capacitor_SMD:C_0805_2012Metric, symbol Device:C
Connections:
- net +3V3: now also C19.1, C20.1
- net GND: now also C19.2, C20.2

Commit message: hw(hardware): decouple the TPL5010 supply pin
U7 (TPL5010) pin 1 VDD carried no local capacitor. Adds C21 100n 0603
beside the module's +3V3 rail entry.

Satisfies the Phase 2.1 deliverable "0.1 uF decoupling cap at the VDD
of every IC" for this device. Unlike U3 this is a compliance gap
rather than a functional risk: the TPL5010 is a nanopower timer and
is not a meaningful transient load.

Separated from the U3 change so either can be reverted alone.

ERC: 0 violations.
Parts:
- added C21: 100n, Capacitor_SMD:C_0603_1608Metric, symbol Device:C
Connections:
- net +3V3: now also C21.2
- net GND: now also C21.1
Changed lines of the file:
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@@
 	)
 	(junction
+		(at 353.06 204.47)
+		(diameter 0)
+		(color 0 0 0 0)
+	)
+	(junction
 		(at 64.77 36.83)
 		(diameter 0)
@@
 	(wire
 		(pts
-			(xy 353.06 203.2) (xy 353.06 207.01)
-		)
-		(stroke
-			(width 0)
-			(type default)
-		)
-	)
-	(wire
-		(pts
 			(xy 363.22 171.45) (xy 360.68 171.45)
 		)
@@
 	(wire
 		(pts
+			(xy 328.93 204.47) (xy 332.74 204.47)
+		)
+		(stroke
+			(width 0)
+			(type default)
+		)
+	)
+	(wire
+		(pts
 			(xy 40.64 251.46) (xy 44.45 251.46)
 		)
@@
 	(wire
 		(pts
+			(xy 340.36 204.47) (xy 353.06 204.47)
+		)
+		(stroke
+			(width 0)
+			(type default)
+		)
+	)
+	(wire
+		(pts
 			(xy 250.19 44.45) (xy 264.16 44.45)
 		)
@@
 	(wire
 		(pts
+			(xy 328.93 208.28) (xy 328.93 204.47)
+		)
+		(stroke
+			(width 0)
+			(type default)
+		)
+	)
+	(wire
+		(pts
 			(xy 121.92 256.54) (xy 127 256.54)
 		)
@@
 	(wire
 		(pts
+			(xy 353.06 204.47) (xy 353.06 207.01)
+		)
+		(stroke
+			(width 0)
+			(type default)
+		)
+	)
+	(wire
+		(pts
 			(xy 26.67 24.13) (xy 27.94 24.13)
 		)
@@
 	(wire
 		(pts
+			(xy 353.06 203.2) (xy 353.06 204.47)
+		)
+		(stroke
+			(width 0)
+			(type default)
+		)
+	)
+	(wire
+		(pts
 			(xy 27.94 24.13) (xy 27.94 26.67)
 		)
@@
 	)
 	(symbol
+		(lib_id "Device:C")
+		(at 336.55 204.47 90)
+		(unit 1)
+		(exclude_from_sim no)
+		(in_bom yes)
+		(on_board yes)
+		(dnp no)
+		(property "Reference" "C21"
+			(at 334.01 198.12 90)
+			(effects
+				(font
+					(size 1.27 1.27)
+				)
+				(justify right)
+			)
+		)
+		(property "Value" "100n"
+			(at 334.01 200.66 90)
+			(effects
+				(font
+					(size 1.27 1.27)
+				)
+				(justify right)
+			)
+		)
+		(property "Footprint" "Capacitor_SMD:C_0603_1608Metric"
+			(at 336.55 203.5048 0)
+			(effects
+				(font
+					(size 1.27 1.27)
+				)
+				(hide yes)
+			)
+		)
+		(property "Datasheet" "~"
+			(at 336.55 204.47 0)
+			(effects
+				(font
+					(size 1.27 1.27)
+				)
+				(hide yes)
+			)
+		)
+		(property "Description" "Unpolarized capacitor"
+			(at 336.55 204.47 0)
+			(effects
+				(font
+					(size 1.27 1.27)
+				)
+				(hide yes)
+			)
+		)
+		(pin "1"
+		)
+		(pin "2"
+		)
+		(instances
+			(project "fortunelabs_mainboard_v0"
+				(path "/1727eecb-65c8-4b57-aa8a-814f366e0831"
+					(reference "C21")
+					(unit 1)
+				)
+			)
+		)
+	)
+	(symbol
 		(lib_id "power:GND")
 		(at 82.55 209.55 0)
@@
 					(unit 1)
 				)
+			)
+		)
+	)
+	(symbol
+		(lib_id "power:GND")
+		(at 328.93 208.28 0)
+		(unit 1)
+		(exclude_from_sim no)
+		(in_bom yes)
+		(on_board yes)
+		(dnp no)
+		(fields_autoplaced yes)
+		(property "Reference" "#PWR036"
+			(at 328.93 214.63 0)
+			(effects
+				(font
+					(size 1.27 1.27)
+				)
+				(hide yes)
+			)
+		)
+		(property "Value" "GND"
+			(at 328.93 213.36 0)
+			(effects
+				(font
+					(size 1.27 1.27)
+				)
+			)
+		)
+		(property "Footprint" ""
+			(at 328.93 208.28 0)
+			(effects
+				(font
+					(size 1.27 1.27)
+				)
+				(hide yes)
+			)
+		)
+		(property "Datasheet" ""
+			(at 328.93 208.28 0)
+			(effects
+				(font
+					(size 1.27 1.27)
+				)
+				(hide yes)
+			)
+		)
+		(property "Description" "Power symbol creates a global label with name \"GND\" , ground"
+			(at 328.93 208.28 0)
+			(effects
+				(font
+					(size 1.27 1.27)
+				)
+				(hide yes)
+			)
+		)
+		(pin "1"
+		)
+		(instances
+			(project "fortunelabs_mainboard_v0"
+				(path "/1727eecb-65c8-4b57-aa8a-814f366e0831"
+					(reference "#PWR036")
+					(unit 1)
+				)
