File: hardware/fortunelabs_mainboard_v0/fortunelabs_mainboard_v0.kicad_sch (KiCad schematic)
At the start: 110 parts, among them J101 Barrel_Jack, J301 USB_C_Receptacle_USB2.0_14P, J401 Micro_SD_Card_Det_Hirose_DM3AT, J701 Conn_02x16_Odd_Even, J801 Conn_02x16_Odd_Even, J901 Conn_02x07_Odd_Even, Q101 AO3401A, SW101 BOOT, SW102 RESET, U101 TPS62162DSG, U201 ESP32-S3-WROOM-2, U501 DS3232M, U601 TPL5010, U701 MCP23017_ML, U801 ADS1115, U802 ADS1115, U901 ULN2803A

Commit message: hw(hardware): shrink the test point drill to 1.0mm
TP1-TP5, TP8 and TP9 move from TestPoint_Plated_Hole_D2.0mm to
TestPoint_THTPad_D2.0mm_Drill1.0mm. The 2.0mm hole was too large; the
pad outer diameter stays 2.0mm, only the drill changes.

TP6 and TP7 keep TestPoint_Loop_D2.50mm_Drill1.0mm_LowProfile. They are
loop points, a different class, and already on a 1.0mm drill.

The exported BOM still names the old footprint and is re-exported in a
commit of its own. No test point footprints are placed on the PCB, so
there is nothing to sync there.
Parts:
- TP1, TP2, TP3, TP4, TP5, TP8, TP9: footprint TestPoint:TestPoint_Plated_Hole_D2.0mm -> TestPoint:TestPoint_THTPad_D2.0mm_Drill1.0mm
Changed lines of the file:
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@@
 			)
 		)
-		(property "Footprint" "TestPoint:TestPoint_Plated_Hole_D2.0mm"
+		(property "Footprint" "TestPoint:TestPoint_THTPad_D2.0mm_Drill1.0mm"
 			(at 74.93 49.53 0)
 			(effects
@@
 			)
 		)
-		(property "Footprint" "TestPoint:TestPoint_Plated_Hole_D2.0mm"
+		(property "Footprint" "TestPoint:TestPoint_THTPad_D2.0mm_Drill1.0mm"
 			(at 262.89 176.53 0)
 			(effects
@@
 			)
 		)
-		(property "Footprint" "TestPoint:TestPoint_Plated_Hole_D2.0mm"
+		(property "Footprint" "TestPoint:TestPoint_THTPad_D2.0mm_Drill1.0mm"
 			(at 252.73 179.07 0)
 			(effects
@@
 			)
 		)
-		(property "Footprint" "TestPoint:TestPoint_Plated_Hole_D2.0mm"
+		(property "Footprint" "TestPoint:TestPoint_THTPad_D2.0mm_Drill1.0mm"
 			(at 151.13 67.31 0)
 			(effects
@@
 			)
 		)
-		(property "Footprint" "TestPoint:TestPoint_Plated_Hole_D2.0mm"
+		(property "Footprint" "TestPoint:TestPoint_THTPad_D2.0mm_Drill1.0mm"
 			(at 29.21 33.02 0)
 			(effects
@@
 			)
 		)
-		(property "Footprint" "TestPoint:TestPoint_Plated_Hole_D2.0mm"
+		(property "Footprint" "TestPoint:TestPoint_THTPad_D2.0mm_Drill1.0mm"
 			(at 264.16 153.67 0)
 			(effects
@@
 			)
 		)
-		(property "Footprint" "TestPoint:TestPoint_Plated_Hole_D2.0mm"
+		(property "Footprint" "TestPoint:TestPoint_THTPad_D2.0mm_Drill1.0mm"
 			(at 184.15 138.43 0)
 			(effects
